Commit message: 安装机械臂

File: description/robot_core.xacro (robot description, xacro)
@@ -14,24 +14,33 @@
         <color rgba="0 0 0 1"/>
     </material>
+    <material name="gray">
+        <color rgba="0.8 0.8 0.8 0.8"/>
+    </material>
     <!-- 基坐标系 base_link -->
     <link name="base_link">
-    </link>
-    <!-- 底板 chassis -->
+        <!--visual>
+            <geometry>
+                <mesh filename="package://panda_sar/meshes/BASE.stl"/>
+            </geometry>
+            <matrial name="black"/>
+        </visual-->
+    </link>
+    <!-- 底盘 UGV01-BASE chassis -->
     <joint name="chassis_joint" type="fixed">
         <parent link="base_link"/>
         <child link="chassis"/>
-        <origin xyz="-0.1 0 0"/>
+        <origin xyz="0 0 0.04656" rpy="0 0 0"/>
     </joint>
     <link name="chassis">
         <visual>
-            <origin xyz="0.15 0 0.075"/>
-            <geometry>
-                <box size="0.3 0.3 0.15"/>
+            <geometry>
+                <box size="0.23146 0.19682 0.09112"/>
             </geometry>
             <material name="white"/>
         </visual>
-        <collision>
-            <geometry>
-                <box size="0.3 0.3 0.15"/>
+        <!-- 碰撞范围 -->
+        <collision>
+            <geometry>
+                <box size="0.23146 0.19682 0.09112"/>
             </geometry>
         </collision>
@@ -41,5 +50,7 @@
         <parent link="base_link"/>
         <child link="left_wheel"/>
-        <origin xyz="0 0.175 0" rpy="-${pi/2} 0 0"/>
+        <!-- Z轴朝外 左翻-->
+        <origin xyz="0 0.12 0.049" rpy="-${pi/2} 0 0"/>
+        <!-- Z轴顺时针为正 -->
         <axis xyz="0 0 1"/>
     </joint>
@@ -61,5 +72,7 @@
         <parent link="base_link"/>
         <child link="right_wheel"/>
-        <origin xyz="0 -0.175 0" rpy="${pi/2} 0 0"/>
+        <!-- Z轴朝外 右翻-->
+        <origin xyz="0 -0.12 0.049" rpy="${pi/2} 0 0"/>
+        <!-- Z轴逆时针为正 -->
         <axis xyz="0 0 -1"/>
     </joint>
@@ -77,17 +90,142 @@
         </collision>
     </link>
-    <!-- 摩擦轮 caster wheel -->
-    <joint name="caster_wheel_joint" type="fixed">
+    <!-- 前进摩擦轮 forward caster wheel -->
+    <joint name="forward_caster_wheel_joint" type="fixed">
         <parent link="chassis"/>
-        <child link="caster_wheel"/>
-        <origin xyz="0.24 0 0"/>
-    </joint>
-    <link name="caster_wheel">
-        <visual>
-            <geometry>
-                <sphere radius="0.05"/>
+        <child link="forward_caster_wheel"/>
+        <origin xyz="0.1 0 -0.04156" rpy="0 0 0"/>
+    </joint>
+    <link name="forward_caster_wheel">
+        <visual>
+            <geometry>
+                <sphere radius="0.01"/>
             </geometry>
             <material name="black"/>
         </visual>
+        <collision>
+            <geometry>
+                <sphere radius="0.01"/>
+            </geometry>
+        </collision>
+    </link>
+    <!-- 后退摩擦轮 backward caster wheel -->
+    <joint name="backward_caster_wheel_joint" type="fixed">
+        <parent link="chassis"/>
+        <child link="backward_caster_wheel"/>
+        <origin xyz="-0.1 0 -0.04156" rpy="0 0 0"/>
+    </joint>
+    <link name="backward_caster_wheel">
+        <visual>
+            <geometry>
+                <sphere radius="0.01"/>
+            </geometry>
+            <material name="black"/>
+        </visual>
+        <collision>
+            <geometry>
+                <sphere radius="0.01"/>
+            </geometry>
+        </collision>
+    </link>
+    <!-- 计算仓 Box -->
+    <joint name="box_joint" type="fixed">
+        <parent link="chassis"/>
+        <child link="llm_box"/>
+        <origin xyz="0 0 0.09056" rpy="0 0 0"/>
+    </joint>
+    <link name="llm_box">
+        <visual>
+            <geometry>
+                <box size="0.085 0.055 0.09"/>
+            </geometry>
+            <material name="white"/>
+        </visual>
+        <collision>
+            <geometry>
+                <box size="0.085 0.055 0.09"/>
+            </geometry>
+        </collision>
+    </link>
+    <!-- 机械臂0级 Base L0  -->
+    <joint name="L0_joint" type="fixed">
+        <parent link="llm_box"/>
+        <child link="L0"/>
+        <origin xyz="0 0 0.132" rpy="0 0 0"/>
+        <axis xyz="0 0 1"/>
+    </joint>
+    <link name="L0" >
+        <visual>
+            <geometry>
+                <mesh filename="package://panda_sar/meshes/L0.stl"/>
+            </geometry>
+            <material name="orange"/>
+        </visual>
+    </link>
+    <!-- 机械臂1级 L1  -->
+    <joint name="L1_joint" type="revolute">
+        <parent link="L0"/>
+        <child link="L1"/>
+        <origin xyz="0 0 0" rpy="0 0 0"/>
+        <axis xyz="0 0 1"/>
+        <limit effort="1000.0" lower="-3.14" upper="3.14" velocity="0.5"/>
+    </joint>
+    <link name="L1" >
+        <visual>
+            <geometry>
+                <mesh filename="package://panda_sar/meshes/L1.stl"/>
+            </geometry>
+            <material name="gray"/>
+        </visual>
+    </link>
+    <!-- 机械臂2级 L2  -->
+    <joint name="L2_joint" type="revolute">
+        <parent link="L1"/>
+        <child link="L2"/>
+        <origin xyz="0 0 0.03796" rpy="0 0 0"/>
+        <axis xyz="0 1 0"/>
+        <limit effort="1000.0" lower="-1.570796" upper="1.570796" velocity="0.5"/>
+    </joint>
+    <link name="L2" >
+        <visual>
+            <origin xyz="0 0 -0.03796" rpy="0 0 0"/>
+            <geometry>
+                <mesh filename="package://panda_sar/meshes/L2.stl"/>
+            </geometry>
+            <material name="orange"/>
+        </visual>
+    </link>
+    <!-- 机械臂3级 L3  -->
+    <joint name="L3_joint" type="revolute">
+        <parent link="L2"/>
+        <child link="L3"/>
+        <origin xyz="0.03 0 0.23682" rpy="0 0 0"/>
+        <axis xyz="0 1 0"/>
+        <limit effort="1000.0" lower="-0.78539815" upper="3.1415926" velocity="0.5"/>
+    </joint>
+    <link name="L3" >
+        <visual>
+            <origin xyz="-0.03 0 -0.27477" rpy="0 0 0"/>
+            <geometry>
+                <mesh filename="package://panda_sar/meshes/L3.stl"/>
+            </geometry>
+            <material name="gray"/>
+        </visual>
+    </link>
+    <!-- 机械臂4级 L4  -->
+    <joint name="L4_joint" type="revolute">
+        <parent link="L3"/>
+        <child link="L4"/>
+        <origin xyz="0 0 0.21599" rpy="0 0 0"/>
+        <axis xyz="0 1 0"/>
+        <limit effort="1000.0" lower="-2.3561942" upper="2.3561942" velocity="0.5"/>
+    </joint>
+    <link name="L4" >
+        <visual>
+            <origin xyz="-0.03 0 -0.49076" rpy="0 0 0"/>
+            <geometry>
+                <mesh filename="package://panda_sar/meshes/L4.stl"/>
+            </geometry>
+            <material name="orange"/>
+        </visual>
     </link>
 </robot>

Commit message: 组装机器人

File: description/robot_core.xacro (robot description, xacro)
@@ -1,5 +1,7 @@
 <?xml version="1.0"?>
 <robot xmlns:xacro="http://www.ros.org/wiki/xacro" >
-    <!-- 定义色彩 define color -->
+    <!-- 引入动惯量 define intertial -->
+    <xacro:include filename="intertial_macros.xacro"/>
+    <!-- 引入 RVIZ 色彩 define rviz color -->
     <material name="white">
         <color rgba="1 1 1 1"/>
@@ -19,10 +21,10 @@
     <!-- 基坐标系 base_link -->
     <link name="base_link">
-        <!--visual>
+        <!-- <visual>
             <geometry>
                 <mesh filename="package://panda_sar/meshes/BASE.stl"/>
             </geometry>
             <matrial name="black"/>
-        </visual-->
+        </visual> -->
     </link>
     <!-- 底盘 UGV01-BASE chassis -->
@@ -33,4 +35,5 @@
     </joint>
     <link name="chassis">
+        <!-- 定义可视物 -->
         <visual>
             <geometry>
@@ -39,5 +42,5 @@
             <material name="white"/>
         </visual>
-        <!-- 碰撞范围 -->
+        <!-- 定义碰撞范围 -->
         <collision>
             <geometry>
@@ -45,5 +48,12 @@
             </geometry>
         </collision>
-    </link>
+        <!-- 定义动惯量 -->
+        <xacro:inertial_box mass="1" x="0.23146" y="0.19682" z="0.09112">
+            <origin xyz="0 0 0" rpy="0 0 0"/>
+        </xacro:inertial_box>
+    </link>
+    <gazebo reference="chassis">
+        <material>Gazebo/Orange</material>
+    </gazebo>
     <!-- 左轮 left wheel -->
     <joint name="left_wheel_joint" type="continuous">
@@ -56,4 +66,5 @@
     </joint>
     <link name="left_wheel">
+        <!-- 定义可视物 -->
         <visual>
             <geometry>
@@ -62,4 +73,5 @@
             <material name="blue"/>
         </visual>
+        <!-- 定义碰撞范围 -->
         <collision>
             <geometry>
@@ -67,5 +79,12 @@
             </geometry>
         </collision>
-    </link>
+        <!-- 定义动惯量 -->
+        <xacro:inertial_cylinder mass="0.1" radius="0.05" length="0.04">
+            <origin xyz="0 0 0" rpy="0 0 0"/>
+        </xacro:inertial_cylinder>
+    </link>
+    <gazebo reference="left_wheel">
+        <material>Gazebo/Blue</material>
+    </gazebo>
     <!-- 右轮 right wheel -->
     <joint name="right_wheel_joint" type="continuous">
@@ -78,4 +97,5 @@
     </joint>
     <link name="right_wheel">
+        <!-- 定义可视物 -->
         <visual>
             <geometry>
@@ -84,4 +104,5 @@
             <material name="blue"/>
         </visual>
+        <!-- 定义碰撞范围 -->
         <collision>
             <geometry>
@@ -89,5 +110,12 @@
             </geometry>
         </collision>
-    </link>
+        <!-- 定义动惯量 -->
+        <xacro:inertial_cylinder mass="0.1" radius="0.05" length="0.04">
+            <origin xyz="0 0 0" rpy="0 0 0"/>
+        </xacro:inertial_cylinder>
+    </link>
+    <gazebo reference="right_wheel">
+        <material>Gazebo/Blue</material>
+    </gazebo>
     <!-- 前进摩擦轮 forward caster wheel -->
     <joint name="forward_caster_wheel_joint" type="fixed">
@@ -97,4 +125,5 @@
     </joint>
     <link name="forward_caster_wheel">
+        <!-- 定义可视物 -->
         <visual>
             <geometry>
@@ -103,4 +132,5 @@
             <material name="black"/>
         </visual>
+        <!-- 定义碰撞范围 -->
         <collision>
             <geometry>
@@ -108,5 +138,14 @@
             </geometry>
         </collision>
-    </link>
+        <!-- 定义动惯量 -->
+        <xacro:inertial_sphere mass="0.1" radius="0.01">
+            <origin xyz="0 0 0" rpy="0 0 0"/>
+        </xacro:inertial_sphere>
+    </link>
+    <gazebo reference="forward_caster_wheel">
+        <material>Gazebo/Black</material>
+        <mu1 value="0.001"/>
+        <mu2 value="0.001"/>
+    </gazebo>
     <!-- 后退摩擦轮 backward caster wheel -->
     <joint name="backward_caster_wheel_joint" type="fixed">
@@ -116,4 +155,5 @@
     </joint>
     <link name="backward_caster_wheel">
+        <!-- 定义可视物 -->
         <visual>
             <geometry>
@@ -122,4 +162,5 @@
             <material name="black"/>
         </visual>
+        <!-- 定义碰撞范围 -->
         <collision>
             <geometry>
@@ -127,5 +168,14 @@
             </geometry>
         </collision>
-    </link>
+        <!-- 定义动惯量 -->
+        <xacro:inertial_sphere mass="0.1" radius="0.01">
+            <origin xyz="0 0 0" rpy="0 0 0"/>
+        </xacro:inertial_sphere>
+    </link>
+    <gazebo reference="backward_caster_wheel">
+        <material>Gazebo/Black</material>
+        <mu1 value="0.001"/>
+        <mu2 value="0.001"/>
+    </gazebo>
     <!-- 计算仓 Box -->
     <joint name="box_joint" type="fixed">
@@ -135,10 +185,12 @@
     </joint>
     <link name="llm_box">
+        <!-- 定义可视物 -->
         <visual>
             <geometry>
                 <box size="0.085 0.055 0.09"/>
             </geometry>
-            <material name="white"/>
-        </visual>
+            <material name="gray"/>
+        </visual>
+        <!-- 定义碰撞范围 -->
         <collision>
             <geometry>
@@ -147,4 +199,7 @@
         </collision>
     </link>
+    <gazebo reference="llm_box">
+        <material>Gazebo/Gray</material>
+    </gazebo>
     <!-- 机械臂0级 Base L0  -->
     <joint name="L0_joint" type="fixed">
@@ -154,12 +209,16 @@
         <axis xyz="0 0 1"/>
     </joint>
-    <link name="L0" >
+    <link name="L0">
+        <!-- 定义可视物 -->
         <visual>
             <geometry>
                 <mesh filename="package://panda_sar/meshes/L0.stl"/>
             </geometry>
-            <material name="orange"/>
-        </visual>
-    </link>
+            <material name="gray"/>
+        </visual>
+    </link>
+    <gazebo reference="L0">
+        <material>Gazebo/Gray</material>
+    </gazebo>
     <!-- 机械臂1级 L1  -->
     <joint name="L1_joint" type="revolute">
@@ -170,5 +229,6 @@
         <limit effort="1000.0" lower="-3.14" upper="3.14" velocity="0.5"/>
     </joint>
-    <link name="L1" >
+    <link name="L1">
+        <!-- 定义可视物 -->
         <visual>
             <geometry>
@@ -178,4 +238,7 @@
         </visual>
     </link>
+    <gazebo reference="L1">
+        <material>Gazebo/Gray</material>
+    </gazebo>
     <!-- 机械臂2级 L2  -->
     <joint name="L2_joint" type="revolute">
@@ -186,5 +249,6 @@
         <limit effort="1000.0" lower="-1.570796" upper="1.570796" velocity="0.5"/>
     </joint>
-    <link name="L2" >
+    <link name="L2">
+        <!-- 定义可视物 -->
         <visual>
             <origin xyz="0 0 -0.03796" rpy="0 0 0"/>
@@ -195,4 +259,7 @@
         </visual>
     </link>
+    <gazebo reference="L2">
+        <material>Gazebo/Orange</material>
+    </gazebo>
     <!-- 机械臂3级 L3  -->
     <joint name="L3_joint" type="revolute">
@@ -203,5 +270,6 @@
         <limit effort="1000.0" lower="-0.78539815" upper="3.1415926" velocity="0.5"/>
     </joint>
-    <link name="L3" >
+    <link name="L3">
+        <!-- 定义可视物 -->
         <visual>
             <origin xyz="-0.03 0 -0.27477" rpy="0 0 0"/>
@@ -212,4 +280,7 @@
         </visual>
     </link>
+    <gazebo reference="L3">
+        <material>Gazebo/Gray</material>
+    </gazebo>
     <!-- 机械臂4级 L4  -->
     <joint name="L4_joint" type="revolute">
@@ -220,5 +291,6 @@
         <limit effort="1000.0" lower="-2.3561942" upper="2.3561942" velocity="0.5"/>
     </joint>
-    <link name="L4" >
+    <link name="L4">
+        <!-- 定义可视物 -->
         <visual>
             <origin xyz="-0.03 0 -0.49076" rpy="0 0 0"/>
@@ -229,3 +301,6 @@
         </visual>
     </link>
+    <gazebo reference="L4">
+        <material>Gazebo/Orange</material>
+    </gazebo>
 </robot>
